Commit message: Update vitirover_gazebo.urdf

File: ROS/vitirover_description/urdf/vitirover_gazebo.urdf (robot description, URDF)
Before this commit: robot differential_wheeled_robot, 8 links, 7 joints
Links:
- removed link hokuyo_link
- added link front_axle, mass 1; collision cylinder length=0.35 radius=0.02; visual cylinder length=0.35 radius=0.02
- link base_footprint: mass 0.0001 -> None; geometry 
- link base_link: mass 5 -> 25; geometry collision box size=0.4 0.8 0.1; visual mesh filename=package://mobile_robot/meshes/chassis.stl scale=10 10 10
- link front_left_wheel: geometry collision cylinder length=0.05 radius=0.088; visual cylinder length=0.05 radius=0.088
- link front_right_wheel: geometry collision cylinder length=0.05 radius=0.088; visual cylinder length=0.05 radius=0.088
- link rear_axle: geometry collision cylinder length=0.35 radius=0.02; visual cylinder length=0.35 radius=0.02
- link rear_left_wheel: geometry collision cylinder length=0.05 radius=0.088; visual cylinder length=0.05 radius=0.088
- link rear_right_wheel: geometry collision cylinder length=0.05 radius=0.088; visual cylinder length=0.05 radius=0.088
Joints:
- removed joint hokuyo_joint
- added joint front_axle_joint: type fixed, parent base_link, child front_axle, origin xyz=0.2 0 0 rpy=4.7124 0 0, axis 0 1 0
- joint base_footprint_joint: origin xyz=0 0 0.04 rpy=0 0 0 -> xyz=0 0 0.1 rpy=0 0 0
- joint front_left_wheel_joint: origin xyz=-0.3 -0.2 0.0 rpy=0 0 0 -> xyz=0.2 -0.1875 0.0 rpy=0 0 0
- joint front_right_wheel_joint: origin xyz=-0.3 0.2 0.0 rpy=0 0 0 -> xyz=0.2 0.1875 0.0 rpy=0 0 0
- joint rear_axle_joint: limit lower=-0.2 upper=0.2 effort=100 velocity=100 -> lower=-0.3142 upper=0.3142 effort=100 velocity=100; origin xyz=0.3 0 0 rpy=1.57079632679 0 0 -> xyz=-0.2 0 0 rpy=4.7124 0 0
- joint rear_left_wheel_axle_joint: origin xyz=0 0 -0.2 rpy=1.57079632679 0 0 -> xyz=0 0 -0.1875 rpy=1.570796 0 0
- joint rear_right_wheel_axle_joint: origin xyz=0 0 0.2 rpy=1.57079632679 0 0 -> xyz=0 0 0.1875 rpy=1.570796 0 0
